File: NCL30160_Demo/NCL30160_Demo.sch (KiCad schematic (older format))
At the start: 18 parts

Commit message: PCB: routing of PCB
Parts:
- removed TP?: VCC, symbol Connector:TestPoint
- removed TP?: GND, symbol Connector:TestPoint
- removed TP?: DIM, symbol Connector:TestPoint
- added C2: 4.7uF, Capacitor_SMD:C_0805_2012Metric, symbol Device:C
- added RV1: R_POT, Potentiometer_SMD:Potentiometer_Bourns_3214J_Horizontal, symbol Device:R_POT
- C1: renamed from C?; value C -> 4.7uF; footprint (none) -> Capacitor_SMD:C_0805_2012Metric
- D1: renamed from D?; footprint (none) -> Diode_SMD:D_SOD-123F
- J1, J2, J3: renamed from J?; footprint (none) -> TCY_connectors:Wire_2_SMD_2x3mm
- L1: renamed from L?; footprint (none) -> Inductor_SMD:L_Taiyo-Yuden_NR-80xx
- R1, R2, R3: renamed from R?; footprint (none) -> Resistor_SMD:R_0603_1608Metric
- R4: renamed from R?; footprint (none) -> Resistor_SMD:R_1206_3216Metric
- TP2, TP3, TP4, TP5: renamed from TP?; footprint (none) -> TestPoint:TestPoint_Pad_D1.0mm
- U1: renamed from U?; symbol TCY_IC:NCL30160 -> NCL30160_Demo-rescue:NCL30160-TCY_IC
Connections:
- net +5V: now also RV1.1, RV1.2; no longer R1.1
- net GND: now also C2.2
- net VCC: now also C2.1
- new net: R1.1, RV1.3
Other:
- moved on the sheet: C1, D1, J1, J2, J3, L1, R1, R2, R3, TP2, TP3
